Commit message: change to depth cam (estimate depth + yaw)

File: detection/install/yolobot_description/share/yolobot_description/robot/yolobot.urdf (robot description, URDF)
Before this commit: robot yolobot, 9 links, 8 joints
Links:
- added link laser_link; visual box size=0.01 0.01 0.01
Joints:
- added joint laser_link_joint: type fixed, parent chassis, child laser_link, origin xyz=0.04 0.0 0.3 rpy=0 0 0

Commit message: finish

File: detection/install/yolobot_description/share/yolobot_description/robot/yolobot.urdf (robot description, URDF)
Before this commit: robot yolobot, 10 links, 9 joints
Links:
- added link laser_link_frame
Joints:
- added joint laser_frame_joint: type fixed, parent laser_link, child laser_link_frame, origin xyz=0.01 0 0 rpy=0 0 0, axis 0 0 0
