Commit message: Add files via upload

File: housem8_robot/housem8_description/robots/mech_urdf/mbse_1jun.urdf (robot description, URDF)
Before this commit: robot mbse, 24 links, 23 joints
Links:
- added link FingerMiddle; visual box size=0.160 0.040 0.080
- link HandCamera: geometry collision box size=0.02 0.08 0.03; visual box size=0.02 0.08 0.03
Joints:
- added joint FingerM: type fixed, parent Hand, child FingerMiddle, origin xyz=-0.0 0.00 0.1 rpy=0.0 1.57 0.0, axis 0.0 1.0 0.0, limit lower=-0.1 upper=0.02 effort=1000.0 velocity=0.5
- joint FingerL: axis 0.0 0.1 0.0 -> 0.0 1.0 0.0; limit lower=-0.02 upper=0.1 effort=1000.0 velocity=0.5 -> lower=-0.025 upper=0.04 effort=1000.0 velocity=0.5
- joint FingerR: limit lower=-0.1 upper=0.02 effort=1000.0 velocity=0.5 -> lower=-0.04 upper=0.025 effort=1000.0 velocity=0.5
