Commit message: name fix

File: housem8_robot/housem8_description/robots/mech_urdf/housem8_master.urdf (robot description, URDF)
Before this commit: robot mbse, 25 links, 24 joints
Links:
- removed link FingerMiddle
- added link TipPoint
Joints:
- removed joint FingerM
- added joint FixedTipJoint: type fixed, parent Hand, child TipPoint, origin xyz=0.0 0.0 0.1 rpy=0.0 0.0 0.0

Commit message: Change End effector position and fix name

File: housem8_robot/housem8_description/robots/mech_urdf/housem8_master.urdf (robot description, URDF)
Before this commit: robot mbse, 25 links, 24 joints
Joints:
- joint FixedTipJoint: origin xyz=0.0 0.0 0.1 rpy=0.0 0.0 0.0 -> xyz=0.0 0.0 0.260 rpy=0.0 0.0 1.570796

Commit message: init

File: housem8_robot/housem8_description/robots/mech_urdf/housem8_master.urdf (robot description, URDF)
Before this commit: robot mbse, 25 links, 24 joints
Links:
- added link base_footprint
Joints:
- removed joint HandGripper
- removed joint LinJ
- removed joint RevJ1
- removed joint RevJ2
- removed joint RevJ3
- removed joint RevJ4
- removed joint RevJ5
- added joint Mani_J0: type prismatic, parent Torsol, child LinearJoint, origin xyz=-0.17 0.0 0.0275 rpy=0.0 0.0 0.0, axis 0.0 0.0 1.0, limit lower=0.0 upper=0.650 effort=1000.0 velocity=10.0
- added joint Mani_J1: type revolute, parent LinearJoint, child Revlink1, origin xyz=0.0 0.0 0.125 rpy=0.0 0.0 3.14, axis 0.0 0.0 1.0, limit lower=-1.3 upper=1.3 effort=1000.0 velocity=0.5
- added joint Mani_J2: type revolute, parent Revlink1, child Revlink2, origin xyz=0.06 0.0 0.05 rpy=0.0 1.57 0.0, axis 0.0 0.0 1.0, limit lower=-1.5 upper=1.5 effort=1000.0 velocity=0.5
- added joint Mani_J3: type revolute, parent Revlink2, child Revlink3, origin xyz=0.0 0.0 0.0 rpy=1.57 1.57 0.0, axis 0.0 0.0 1.0, limit lower=-1.2 upper=2.0 effort=1000.0 velocity=0.5
- added joint Mani_J4: type revolute, parent Revlink3, child Revlink4, origin xyz=-0.350 0.0 0.0 rpy=0.0 0.0 0.0, axis 0.0 0.0 1.0, limit lower=-1.9 upper=1.9 effort=1000.0 velocity=0.5
- added joint Mani_J5: type revolute, parent Revlink4, child Revlink5, origin xyz=-0.331 0.0 -0.0 rpy=0.0 0.0 0.0, axis 0.0 0.0 1.0, limit lower=-3.14 upper=3.14 effort=1000.0 velocity=0.5
- added joint Mani_J6: type revolute, parent Revlink5, child Hand, origin xyz=-0.05 -0.0 -0.0 rpy=0.0 -1.57 0.0, axis 0.0 0.0 1.0, limit lower=-3.14 upper=3.14 effort=1000.0 velocity=0.5
