Commit message: rerun msa

File: housem8_robot/housem8_description/robots/housem8.ros1_control.xacro (robot description, xacro)
@@ -1,80 +1,110 @@
 <?xml version='1.0' encoding='utf-8'?>
 <robot xmlns:xacro="http://www.ros.org/wiki/xacro" name="housem8">
-    <transmission name="trans_BodyCam">
+    <transmission name="trans_wheel_right_joint">
         <type>transmission_interface/SimpleTransmission</type>
-        <joint name="BodyCam">
+        <joint name="wheel_right_joint">
+            <hardwareInterface>hardware_interface/EffortJointInterface</hardwareInterface>
+        </joint>
+        <actuator name="wheel_right_joint_motor">
+            <hardwareInterface>hardware_interface/EffortJointInterface</hardwareInterface>
+            <mechanicalReduction>1</mechanicalReduction>
+        </actuator>
+    </transmission>
+    <transmission name="trans_wheel_left_joint">
+        <type>transmission_interface/SimpleTransmission</type>
+        <joint name="wheel_left_joint">
+            <hardwareInterface>hardware_interface/EffortJointInterface</hardwareInterface>
+        </joint>
+        <actuator name="wheel_left_joint_motor">
+            <hardwareInterface>hardware_interface/EffortJointInterface</hardwareInterface>
+            <mechanicalReduction>1</mechanicalReduction>
+        </actuator>
+    </transmission>
+    <transmission name="trans_Casterwheel_left_joint">
+        <type>transmission_interface/SimpleTransmission</type>
+        <joint name="Casterwheel_left_joint">
+            <hardwareInterface>hardware_interface/EffortJointInterface</hardwareInterface>
+        </joint>
+        <actuator name="Casterwheel_left_joint_motor">
+            <hardwareInterface>hardware_interface/EffortJointInterface</hardwareInterface>
+            <mechanicalReduction>1</mechanicalReduction>
+        </actuator>
+    </transmission>
+    <transmission name="trans_Casterwheel_right_joint">
+        <type>transmission_interface/SimpleTransmission</type>
+        <joint name="Casterwheel_right_joint">
+            <hardwareInterface>hardware_interface/EffortJointInterface</hardwareInterface>
+        </joint>
+        <actuator name="Casterwheel_right_joint_motor">
+            <hardwareInterface>hardware_interface/EffortJointInterface</hardwareInterface>
+            <mechanicalReduction>1</mechanicalReduction>
+        </actuator>
+    </transmission>
+    <transmission name="trans_Mani_J0">
+        <type>transmission_interface/SimpleTransmission</type>
+        <joint name="Mani_J0">
             <hardwareInterface>hardware_interface/PositionJointInterface</hardwareInterface>
         </joint>
-        <actuator name="BodyCam_motor">
+        <actuator name="Mani_J0_motor">
             <hardwareInterface>hardware_interface/PositionJointInterface</hardwareInterface>
             <mechanicalReduction>1</mechanicalReduction>
         </actuator>
     </transmission>
-    <transmission name="trans_LinJ">
+    <transmission name="trans_Mani_J1">
         <type>transmission_interface/SimpleTransmission</type>
-        <joint name="LinJ">
+        <joint name="Mani_J1">
             <hardwareInterface>hardware_interface/PositionJointInterface</hardwareInterface>
         </joint>
-        <actuator name="LinJ_motor">
+        <actuator name="Mani_J1_motor">
             <hardwareInterface>hardware_interface/PositionJointInterface</hardwareInterface>
             <mechanicalReduction>1</mechanicalReduction>
         </actuator>
     </transmission>
-    <transmission name="trans_RevJ1">
+    <transmission name="trans_Mani_J2">
         <type>transmission_interface/SimpleTransmission</type>
-        <joint name="RevJ1">
+        <joint name="Mani_J2">
             <hardwareInterface>hardware_interface/PositionJointInterface</hardwareInterface>
         </joint>
-        <actuator name="RevJ1_motor">
+        <actuator name="Mani_J2_motor">
             <hardwareInterface>hardware_interface/PositionJointInterface</hardwareInterface>
             <mechanicalReduction>1</mechanicalReduction>
         </actuator>
     </transmission>
-    <transmission name="trans_RevJ2">
+    <transmission name="trans_Mani_J3">
         <type>transmission_interface/SimpleTransmission</type>
-        <joint name="RevJ2">
+        <joint name="Mani_J3">
             <hardwareInterface>hardware_interface/PositionJointInterface</hardwareInterface>
         </joint>
-        <actuator name="RevJ2_motor">
+        <actuator name="Mani_J3_motor">
             <hardwareInterface>hardware_interface/PositionJointInterface</hardwareInterface>
             <mechanicalReduction>1</mechanicalReduction>
         </actuator>
     </transmission>
-    <transmission name="trans_RevJ3">
+    <transmission name="trans_Mani_J4">
         <type>transmission_interface/SimpleTransmission</type>
-        <joint name="RevJ3">
+        <joint name="Mani_J4">
             <hardwareInterface>hardware_interface/PositionJointInterface</hardwareInterface>
         </joint>
-        <actuator name="RevJ3_motor">
+        <actuator name="Mani_J4_motor">
             <hardwareInterface>hardware_interface/PositionJointInterface</hardwareInterface>
             <mechanicalReduction>1</mechanicalReduction>
         </actuator>
     </transmission>
-    <transmission name="trans_RevJ4">
+    <transmission name="trans_Mani_J5">
         <type>transmission_interface/SimpleTransmission</type>
-        <joint name="RevJ4">
+        <joint name="Mani_J5">
             <hardwareInterface>hardware_interface/PositionJointInterface</hardwareInterface>
         </joint>
-        <actuator name="RevJ4_motor">
+        <actuator name="Mani_J5_motor">
             <hardwareInterface>hardware_interface/PositionJointInterface</hardwareInterface>
             <mechanicalReduction>1</mechanicalReduction>
         </actuator>
     </transmission>
-    <transmission name="trans_RevJ5">
+    <transmission name="trans_Mani_J6">
         <type>transmission_interface/SimpleTransmission</type>
-        <joint name="RevJ5">
+        <joint name="Mani_J6">
             <hardwareInterface>hardware_interface/PositionJointInterface</hardwareInterface>
         </joint>
-        <actuator name="RevJ5_motor">
-            <hardwareInterface>hardware_interface/PositionJointInterface</hardwareInterface>
-            <mechanicalReduction>1</mechanicalReduction>
-        </actuator>
-    </transmission>
-    <transmission name="trans_HandGripper">
-        <type>transmission_interface/SimpleTransmission</type>
-        <joint name="HandGripper">
-            <hardwareInterface>hardware_interface/PositionJointInterface</hardwareInterface>
-        </joint>
-        <actuator name="HandGripper_motor">
+        <actuator name="Mani_J6_motor">
             <hardwareInterface>hardware_interface/PositionJointInterface</hardwareInterface>
             <mechanicalReduction>1</mechanicalReduction>
