Commit message: Update Xarco again

File: housem8_robot/housem8_description/robots/housem8.gazebo.xacro (robot description, xacro)
@@ -166,6 +166,6 @@
             <ros>
                 <namespace>/housem8</namespace>
-                <argument>/cmd_vel:=cmd_vel</argument>
-                <argument>/odom:=odom</argument>
+                <argument>-r ~/cmd_vel:=cmd_vel</argument>
+                <argument>-r ~/odom:=odom</argument>
             </ros>
             <publish_odom>true</publish_odom>

File: housem8_robot/housem8_description/robots/housem8.ros2_control.xacro (robot description, xacro)
@@ -20,21 +20,9 @@
         <xacro:configure_joint joint_name="Mani_J5" initial_position="0.0"/>
         <xacro:configure_joint joint_name="Mani_J6" initial_position="0.0"/>
-        <!-- <xacro:configure_joint joint_name="wheel_left_joint" initial_position="0.0"/>
-        <xacro:configure_joint joint_name="wheel_right_joint" initial_position="0.0"/> -->
-        <!-- <joint name="wheel_left_joint">
-          <command_interface name="velocity">
-          </command_interface>
-          <state_interface name="position"/>
-          <state_interface name="velocity"/>
-        </joint>
-        <joint name="wheel_right_joint">
-          <command_interface name="velocity">
-          </command_interface>
-          <state_interface name="position"/>
-          <state_interface name="velocity"/>
-        </joint> -->
+        <xacro:configure_joint joint_name="FingerR" initial_position="0.0"/>
+        <xacro:configure_joint joint_name="FingerL" initial_position="0.0"/>
       </ros2_control>
     <gazebo>
-      <plugin filename="libgazebo_ros2_control.so" name="gazebo_ros2_control">
+      <plugin filename="libgazebo_ros2_control.so" name="gazebo_ros2_control_arm">
         <parameters>$(find housem8_description)/config/housem8_ros_controllers.yaml</parameters>
       </plugin>

Commit message: Add files via upload

File: housem8_robot/housem8_description/robots/housem8.gazebo.xacro (robot description, xacro)
@@ -38,5 +38,5 @@
                 <slip1>0</slip1>
                 <slip2>0</slip2>
-                <material>Gazebo/Blue</material>
+                <material>Gazebo/Blue</material> /housem8/cmd_vel
             </gazebo>
         </xacro:macro>
@@ -51,5 +51,5 @@
         <xacro:base link="CasterCase_Right"/>
         <!-- <xacro:base link="CasterWheel_Right"/> -->
-        <xacro:base link="mobilebaseIII"/>
+        <xacro:base link="mobilebaseIII"/> /housem8/cmd_vel
         <xacro:base link="mobilebaseIV"/>
         <xacro:base link="Lidar_Front"/>
@@ -73,5 +73,5 @@
         <update_rate>10.0</update_rate>
         <camera name="camera">
-            <pose>0 0 0 0 0 0</pose>
+            <pose>0 0 0 0 0 3.14</pose>
             <horizontal_fov>1.3962634</horizontal_fov>
             <image>
@@ -103,5 +103,5 @@
         <update_rate>10.0</update_rate>
         <camera name="camera">
-            <pose>0 0 0 0 0 0</pose>
+            <pose>0 0 0 -3.14 -1.57 3.14</pose>
             <horizontal_fov>1.3962634</horizontal_fov>
             <image>

File: housem8_robot/housem8_description/robots/housem8.xacro (robot description, xacro)
@@ -667,5 +667,5 @@
     <link name='rgb_cam_camera_link'/>
     <joint name="rgb_cam_camera_link_joint" type="fixed">
-		<origin rpy="0 0 0" xyz="0.04 0.0 0.2"/>
+		<origin rpy="0 0 0" xyz="0.0 0.0 0."/>
 		<parent link="TorsolCamera"/>
 		<child link="rgb_cam_camera_link"/>
@@ -673,5 +673,5 @@
     <link name="rgb_cam_camera_link_frame"/>
     <joint name="rgb_cam_camera_frame_joint" type="fixed">
-        <origin xyz="0.01 0 0" rpy="0 0 0" />
+        <origin xyz="0.0 0 0.0" rpy="0 0 0" />
         <parent link="rgb_cam_camera_link" />
         <child link="rgb_cam_camera_link_frame" />
@@ -680,5 +680,5 @@
     <link name='rgb_hand_cam_camera_link'/>
     <joint name="rgb_hand_cam_camera_link_joint" type="fixed">
-		<origin rpy="0 0 0" xyz="0.04 0.0 0.2"/>
+		<origin rpy="0 0 0" xyz="0 0 0"/>
 		<parent link="HandCamera"/>
 		<child link="rgb_hand_cam_camera_link"/>
@@ -686,5 +686,5 @@
     <link name="rgb_hand_cam_camera_link_frame"/>
     <joint name="rgb_hand_cam_camera_frame_joint" type="fixed">
-        <origin xyz="0.01 0 0" rpy="0 0 0" />
+        <origin xyz="0 0 0" rpy="0 0 0" />
         <parent link="rgb_hand_cam_camera_link" />
         <child link="rgb_hand_cam_camera_link_frame" />

Commit message: Add files via upload

File: housem8_robot/housem8_description/robots/housem8.gazebo.xacro (robot description, xacro)
@@ -67,5 +67,5 @@
         <xacro:arm_gazebo link="Hand"/>
     </xacro:macro>
-    <!-- Body Camera -->
+   <!-- Body Camera -->
     <gazebo reference="rgb_cam_camera_link_frame">
         <sensor type="depth" name="rgb_cam">
@@ -73,5 +73,5 @@
         <update_rate>10.0</update_rate>
         <camera name="camera">
-            <pose>0 0 0 0 0 0</pose>
+            <pose>0 0 0 0 0 3.14</pose>
             <horizontal_fov>1.3962634</horizontal_fov>
             <image>
@@ -103,5 +103,5 @@
         <update_rate>10.0</update_rate>
         <camera name="camera">
-            <pose>0 0 0 0 0 0</pose>
+            <pose>0 0 0 -3.14 -1.57 3.14</pose>
             <horizontal_fov>1.3962634</horizontal_fov>
             <image>
@@ -156,14 +156,14 @@
         <plugin name='diff_drive' filename="libgazebo_ros_diff_drive.so">
             <alwaysOn>true</alwaysOn>
-            <updateRate>10</updateRate>
+            <updateRate>2000</updateRate>
             <left_joint>wheel_left_joint</left_joint>
             <right_joint>wheel_right_joint</right_joint>
             <wheel_separation>0.380</wheel_separation>
             <wheel_diameter>0.200</wheel_diameter>
-            <max_wheel_torque>5.0</max_wheel_torque>
-            <max_wheel_acceleration>5.0</max_wheel_acceleration>
+            <max_wheel_torque>50.0</max_wheel_torque>
+            <max_wheel_acceleration>20.0</max_wheel_acceleration>
             <commandTopic>cmd_vel</commandTopic>
             <ros>
-                <namespace>/housem8</namespace>
+                <namespace>/</namespace>
                 <argument>-r ~/cmd_vel:=cmd_vel</argument>
                 <argument>-r ~/odom:=odom</argument>
@@ -205,5 +205,6 @@
                 <plugin name="lidar_controller" filename="libgazebo_ros_ray_sensor.so">
                     <ros>
-                        <remapping>~/out:=/housem8/scan/front</remapping>
+                        <!-- <remapping>~/out:=/housem8/scan/front</remapping> -->
+                        <remapping>~/out:=/scan</remapping>
                       </ros>
                     <output_type>sensor_msgs/LaserScan</output_type>

File: housem8_robot/housem8_description/robots/housem8.ros1_control.xacro (robot description, xacro)
@@ -1,110 +1,80 @@
 <?xml version='1.0' encoding='utf-8'?>
 <robot xmlns:xacro="http://www.ros.org/wiki/xacro" name="housem8">
-    <transmission name="trans_wheel_right_joint">
+    <transmission name="trans_BodyCam">
         <type>transmission_interface/SimpleTransmission</type>
-        <joint name="wheel_right_joint">
-            <hardwareInterface>hardware_interface/EffortJointInterface</hardwareInterface>
-        </joint>
-        <actuator name="wheel_right_joint_motor">
-            <hardwareInterface>hardware_interface/EffortJointInterface</hardwareInterface>
-            <mechanicalReduction>1</mechanicalReduction>
-        </actuator>
-    </transmission>
-    <transmission name="trans_wheel_left_joint">
-        <type>transmission_interface/SimpleTransmission</type>
-        <joint name="wheel_left_joint">
-            <hardwareInterface>hardware_interface/EffortJointInterface</hardwareInterface>
-        </joint>
-        <actuator name="wheel_left_joint_motor">
-            <hardwareInterface>hardware_interface/EffortJointInterface</hardwareInterface>
-            <mechanicalReduction>1</mechanicalReduction>
-        </actuator>
-    </transmission>
-    <transmission name="trans_Casterwheel_left_joint">
-        <type>transmission_interface/SimpleTransmission</type>
-        <joint name="Casterwheel_left_joint">
-            <hardwareInterface>hardware_interface/EffortJointInterface</hardwareInterface>
-        </joint>
-        <actuator name="Casterwheel_left_joint_motor">
-            <hardwareInterface>hardware_interface/EffortJointInterface</hardwareInterface>
-            <mechanicalReduction>1</mechanicalReduction>
-        </actuator>
-    </transmission>
-    <transmission name="trans_Casterwheel_right_joint">
-        <type>transmission_interface/SimpleTransmission</type>
-        <joint name="Casterwheel_right_joint">
-            <hardwareInterface>hardware_interface/EffortJointInterface</hardwareInterface>
-        </joint>
-        <actuator name="Casterwheel_right_joint_motor">
-            <hardwareInterface>hardware_interface/EffortJointInterface</hardwareInterface>
-            <mechanicalReduction>1</mechanicalReduction>
-        </actuator>
-    </transmission>
-    <transmission name="trans_Mani_J0">
-        <type>transmission_interface/SimpleTransmission</type>
-        <joint name="Mani_J0">
+        <joint name="BodyCam">
             <hardwareInterface>hardware_interface/PositionJointInterface</hardwareInterface>
         </joint>
-        <actuator name="Mani_J0_motor">
+        <actuator name="BodyCam_motor">
             <hardwareInterface>hardware_interface/PositionJointInterface</hardwareInterface>
             <mechanicalReduction>1</mechanicalReduction>
         </actuator>
     </transmission>
-    <transmission name="trans_Mani_J1">
+    <transmission name="trans_LinJ">
         <type>transmission_interface/SimpleTransmission</type>
-        <joint name="Mani_J1">
+        <joint name="LinJ">
             <hardwareInterface>hardware_interface/PositionJointInterface</hardwareInterface>
         </joint>
-        <actuator name="Mani_J1_motor">
+        <actuator name="LinJ_motor">
             <hardwareInterface>hardware_interface/PositionJointInterface</hardwareInterface>
             <mechanicalReduction>1</mechanicalReduction>
         </actuator>
     </transmission>
-    <transmission name="trans_Mani_J2">
+    <transmission name="trans_RevJ1">
         <type>transmission_interface/SimpleTransmission</type>
-        <joint name="Mani_J2">
+        <joint name="RevJ1">
             <hardwareInterface>hardware_interface/PositionJointInterface</hardwareInterface>
         </joint>
-        <actuator name="Mani_J2_motor">
+        <actuator name="RevJ1_motor">
             <hardwareInterface>hardware_interface/PositionJointInterface</hardwareInterface>
             <mechanicalReduction>1</mechanicalReduction>
         </actuator>
     </transmission>
-    <transmission name="trans_Mani_J3">
+    <transmission name="trans_RevJ2">
         <type>transmission_interface/SimpleTransmission</type>
-        <joint name="Mani_J3">
+        <joint name="RevJ2">
             <hardwareInterface>hardware_interface/PositionJointInterface</hardwareInterface>
         </joint>
-        <actuator name="Mani_J3_motor">
+        <actuator name="RevJ2_motor">
             <hardwareInterface>hardware_interface/PositionJointInterface</hardwareInterface>
             <mechanicalReduction>1</mechanicalReduction>
         </actuator>
     </transmission>
-    <transmission name="trans_Mani_J4">
+    <transmission name="trans_RevJ3">
         <type>transmission_interface/SimpleTransmission</type>
-        <joint name="Mani_J4">
+        <joint name="RevJ3">
             <hardwareInterface>hardware_interface/PositionJointInterface</hardwareInterface>
         </joint>
-        <actuator name="Mani_J4_motor">
+        <actuator name="RevJ3_motor">
             <hardwareInterface>hardware_interface/PositionJointInterface</hardwareInterface>
             <mechanicalReduction>1</mechanicalReduction>
         </actuator>
     </transmission>
-    <transmission name="trans_Mani_J5">
+    <transmission name="trans_RevJ4">
         <type>transmission_interface/SimpleTransmission</type>
-        <joint name="Mani_J5">
+        <joint name="RevJ4">
             <hardwareInterface>hardware_interface/PositionJointInterface</hardwareInterface>
         </joint>
-        <actuator name="Mani_J5_motor">
+        <actuator name="RevJ4_motor">
             <hardwareInterface>hardware_interface/PositionJointInterface</hardwareInterface>
             <mechanicalReduction>1</mechanicalReduction>
         </actuator>
     </transmission>
-    <transmission name="trans_Mani_J6">
+    <transmission name="trans_RevJ5">
         <type>transmission_interface/SimpleTransmission</type>
-        <joint name="Mani_J6">
+        <joint name="RevJ5">
             <hardwareInterface>hardware_interface/PositionJointInterface</hardwareInterface>
         </joint>
-        <actuator name="Mani_J6_motor">
+        <actuator name="RevJ5_motor">
+            <hardwareInterface>hardware_interface/PositionJointInterface</hardwareInterface>
+            <mechanicalReduction>1</mechanicalReduction>
+        </actuator>
+    </transmission>
+    <transmission name="trans_HandGripper">
+        <type>transmission_interface/SimpleTransmission</type>
+        <joint name="HandGripper">
+            <hardwareInterface>hardware_interface/PositionJointInterface</hardwareInterface>
+        </joint>
+        <actuator name="HandGripper_motor">
             <hardwareInterface>hardware_interface/PositionJointInterface</hardwareInterface>
             <mechanicalReduction>1</mechanicalReduction>

File: housem8_robot/housem8_description/robots/housem8.xacro (robot description, xacro)
@@ -2,4 +2,5 @@
 <robot xmlns:xacro="http://www.ros.org/wiki/xacro" name="housem8">
     <link name="base_footprint">
+        <origin xyz="0.0 0.0 0.0" rpy="0.0 0.0 3.14" />
     </link>
     <link name="mobilebaseI">
@@ -14,5 +15,5 @@
         </visual>
         <inertial>
-            <mass value="10.0"/>
+            <mass value="20.0"/>
             <inertia ixx="0.3" ixy="0.0" ixz="0.0"
                      iyy="0.3" iyz="0.0" izz="0.3"/>
@@ -28,5 +29,5 @@
         <parent link="base_footprint"/>
         <child link="mobilebaseI"/>
-        <origin rpy="0 0 0" xyz="0 0 0"/>
+        <origin rpy="0 0 3.14" xyz="0 0 0"/>
     </joint>
     <link name="mobilebaseII">
@@ -667,5 +668,5 @@
     <link name='rgb_cam_camera_link'/>
     <joint name="rgb_cam_camera_link_joint" type="fixed">
-		<origin rpy="0 0 0" xyz="0.04 0.0 0.2"/>
+		<origin rpy="0 0 0" xyz="0 0 0"/>
 		<parent link="TorsolCamera"/>
 		<child link="rgb_cam_camera_link"/>
@@ -673,5 +674,5 @@
     <link name="rgb_cam_camera_link_frame"/>
     <joint name="rgb_cam_camera_frame_joint" type="fixed">
-        <origin xyz="0.01 0 0" rpy="0 0 0" />
+        <origin xyz="0 0 0" rpy="0 0 0" />
         <parent link="rgb_cam_camera_link" />
         <child link="rgb_cam_camera_link_frame" />
@@ -680,5 +681,5 @@
     <link name='rgb_hand_cam_camera_link'/>
     <joint name="rgb_hand_cam_camera_link_joint" type="fixed">
-		<origin rpy="0 0 0" xyz="0.04 0.0 0.2"/>
+		<origin rpy="0 0 0" xyz="0.0 0.0 0.0"/>
 		<parent link="HandCamera"/>
 		<child link="rgb_hand_cam_camera_link"/>
@@ -686,5 +687,5 @@
     <link name="rgb_hand_cam_camera_link_frame"/>
     <joint name="rgb_hand_cam_camera_frame_joint" type="fixed">
-        <origin xyz="0.01 0 0" rpy="0 0 0" />
+        <origin xyz="0  0 0" rpy="0 0 0" />
         <parent link="rgb_hand_cam_camera_link" />
         <child link="rgb_hand_cam_camera_link_frame" />

File: housem8_robot/housem8_description/robots/housem8_ros1.urdf.xacro (robot description, xacro)
@@ -1,5 +1,5 @@
 <?xml version='1.0' encoding='utf-8'?>
 <robot xmlns:xacro="http://www.ros.org/wiki/xacro" name="housem8">
-  <xacro:include filename="$(find housem8_manipulator_server)/../../../housem8_robot/housem8_description/robots/housem8.xacro"/>
+  <xacro:include filename="$(find housem8_manipulator_server)/../../../housem8_robot/housem8_description/robots/housem8.xarco"/>
   <xacro:include filename="$(find housem8_manipulator_server)/../../../housem8_robot/housem8_description/robots/housem8.ros1_control.xacro"/>
 </robot>
